File: ICS-43434-PCB.kicad_pcb (KiCad board)
At the start: 2 copper layers, 11.3 x 11.3 mm, 5 parts, among them J1 Conn_01x03, J2 Conn_01x03

Commit message: minor adjustments
Parts:
- removed J1, J2: Conn_01x03, Connector_PinHeader_2.54mm:PinHeader_1x03_P2.54mm_Vertical
- added TP1: +, Connector_PinHeader_2.54mm:PinHeader_1x01_P2.54mm_Vertical, F.Cu at (96.6, 101.2)
- added TP2: SC, Connector_PinHeader_2.54mm:PinHeader_1x01_P2.54mm_Vertical, F.Cu at (98.5, 96.5)
- added TP3: LR, Connector_PinHeader_2.54mm:PinHeader_1x01_P2.54mm_Vertical, F.Cu at (101.3, 96.7)
- added TP4: WS, Connector_PinHeader_2.54mm:PinHeader_1x01_P2.54mm_Vertical, F.Cu at (103.1, 98.2)
- added TP5: SD, Connector_PinHeader_2.54mm:PinHeader_1x01_P2.54mm_Vertical, F.Cu at (103.5, 100.6)
- added TP6: -, Connector_PinHeader_2.54mm:PinHeader_1x01_P2.54mm_Vertical, F.Cu at (96.7, 98.5)
- moved C1 41.6 mm to (98.2, 103.8), turned to 180 degrees
- moved MK1 37.3 mm to (100.0, 100.7)
- moved R1 35.6 mm to (101.8, 103.8), turned to 0 degrees
Routing:
- net GND: track 20.3 -> 0.98 mm, vias 2 -> 1
- net +3V3: track 11.6 -> 4.54 mm, vias 1 -> 0
- net SCK: track 2.91 -> 4.80 mm
- net WS: track 3.37 -> 4.84 mm
- added copper zone on B.Cu, net GND
- added copper zone on F.Cu, net GND
Other:
- board text added: "ICS43434 v1"
