File: ICS-43434-PCB.sch (KiCad schematic (older format))
At the start: 5 parts, among them J1 Conn_01x03, J2 Conn_01x03

Commit message: minor adjustments
Parts:
- removed J1, J2: Conn_01x03, Connector_PinHeader_2.54mm:PinHeader_1x03_P2.54mm_Vertical, symbol Connector_Generic:Conn_01x03
- added TP1: VDD, Connector_PinHeader_2.54mm:PinHeader_1x01_P2.54mm_Vertical, symbol Connector:TestPoint
- added TP2: SCK, Connector_PinHeader_2.54mm:PinHeader_1x01_P2.54mm_Vertical, symbol Connector:TestPoint
- added TP3: LR, Connector_PinHeader_2.54mm:PinHeader_1x01_P2.54mm_Vertical, symbol Connector:TestPoint
- added TP4: WS, Connector_PinHeader_2.54mm:PinHeader_1x01_P2.54mm_Vertical, symbol Connector:TestPoint
- added TP5: SD, Connector_PinHeader_2.54mm:PinHeader_1x01_P2.54mm_Vertical, symbol Connector:TestPoint
- added TP6: GND, Connector_PinHeader_2.54mm:PinHeader_1x01_P2.54mm_Vertical, symbol Connector:TestPoint
Connections:
- net +3V3: now also TP1.1
- net GND: now also TP6.1
- net LR: now also TP3.1
- net SCK: now also TP2.1
- net SD: now also TP5.1
- net WS: now also TP4.1
Other:
- moved on the sheet: C1, MK1, R1
